Commit message: fix<mini_4wd>: 修复仿真失败的问题

File: models/mini_4wd/urdf/all.xacro (robot description, xacro)
@@ -26,7 +26,7 @@
   <xacro:property name="box_mass" value="0.6" />
   <xacro:property name="model_name" value="mini_4wd" />
-  <xacro:property name="model_dir" value="$(find ugv_ctrl)/models/${model_name}" />
+  <xacro:property name="model_dir" value="$(find ugv_descriptions)/models/${model_name}" />
   <xacro:property name="urdf_dir" value="${model_dir}/urdf" />
-  <xacro:property name="mesh_dir" value="package://ugv_ctrl/models/mini_4wd/meshes" />
+  <xacro:property name="mesh_dir" value="package://ugv_descriptions/models/mini_4wd/meshes" />
   <xacro:macro name="box_inertial_matrix" params="m w h d">
     <inertial>

File: models/mini_4wd/urdf/gazebo.xacro (robot description, xacro)
@@ -7,12 +7,17 @@
     </plugin>
     <plugin
-      filename="gz-sim-joint-state-publisher-system"
-      name="gz::sim::systems::JointStatePublisher">
-    </plugin>
-    <plugin
       filename="gz-sim-odometry-publisher-system"
       name="gz::sim::systems::OdometryPublisher">
       <odom_frame>odom</odom_frame>
       <robot_base_frame>base_link</robot_base_frame>
+    </plugin>
+    <plugin
+      filename="gz-sim-sensors-system"
+      name="gz::sim::systems::Sensors">
+      <render_engine>ogre2</render_engine>
+    </plugin>
+    <plugin
+      filename="gz-sim-imu-system"
+      name="gz::sim::systems::Imu">
     </plugin>
   </gazebo>
